File: KiCAD/Antilog_NPNO_PCB/Antilog_NPNO_PCB.sch (KiCad schematic (older format))
At the start: 38 parts, among them J1 PWR_IN, J2 TP_GND, J3 Couarse, J4 Modulation, J5 Master_Out, J6 I_REF, J7 I_Sink, Q1 2SC1815, Q2 2SC1815, U1 TL072

Commit message: implementation Test
Parts:
- added H1, H2, H3, H4: MountingHole, MountingHole:MountingHole_3.2mm_M3, symbol Mechanical:MountingHole
Connections:
- net GND: now also U1.3 (+), U1.5 (+); no longer U1.3 (+), U1.5 (+)
- net at R11.1, RV4.1, RV4.2: now also U1.7; no longer U1.1
- net at R10.2, R11.2, R7.1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: now also U1.6 (-); no longer U1.2 (-)
- net at C5.2, Q1.2 (C), R14.2: now also U1.2 (-); no longer U1.6 (-)
- net at C5.1, R15.2: now also U1.1; no longer U1.7
Changed lines of the file:
@@
 $Comp
 L Amplifier_Operational:TL072 U1
-U 1 1 5F8E2874
+U 2 1 5F8E2874
 P 6550 3950
 F 0 "U1" H 6200 4350 50  0000 C CNN
@@
 F 2 "Package_DIP:DIP-8_W7.62mm_Socket" H 6550 3950 50  0001 C CNN
 F 3 "http://www.ti.com/lit/ds/symlink/tl071.pdf" H 6550 3950 50  0001 C CNN
-	1    6550 3950
+	2    6550 3950
 	1    0    0    -1
 $EndComp
@@
 $Comp
 L Amplifier_Operational:TL072 U1
-U 2 1 5F8E9E6F
+U 1 1 5F8E9E6F
 P 8600 4900
 F 0 "U1" H 8600 5267 50  0000 C CNN
@@
 F 2 "Package_DIP:DIP-8_W7.62mm_Socket" H 8600 4900 50  0001 C CNN
 F 3 "http://www.ti.com/lit/ds/symlink/tl071.pdf" H 8600 4900 50  0001 C CNN
-	2    8600 4900
+	1    8600 4900
 	1    0    0    -1
 $EndComp
@@
 Wire Wire Line
 	4750 3600 4750 3550
+$Comp
+L Mechanical:MountingHole H1
+U 1 1 5F938EE3
+P 2250 6000
+F 0 "H1" H 2350 6046 50  0000 L CNN
+F 1 "MountingHole" H 2350 5955 50  0000 L CNN
+F 2 "MountingHole:MountingHole_3.2mm_M3" H 2250 6000 50  0001 C CNN
+F 3 "~" H 2250 6000 50  0001 C CNN
+	1    2250 6000
+	1    0    0    -1
+$EndComp
+$Comp
+L Mechanical:MountingHole H2
+U 1 1 5F939774
+P 2250 6300
+F 0 "H2" H 2350 6346 50  0000 L CNN
+F 1 "MountingHole" H 2350 6255 50  0000 L CNN
+F 2 "MountingHole:MountingHole_3.2mm_M3" H 2250 6300 50  0001 C CNN
+F 3 "~" H 2250 6300 50  0001 C CNN
+	1    2250 6300
+	1    0    0    -1
+$EndComp
+$Comp
+L Mechanical:MountingHole H3
+U 1 1 5F93B327
+P 2250 6600
+F 0 "H3" H 2350 6646 50  0000 L CNN
+F 1 "MountingHole" H 2350 6555 50  0000 L CNN
+F 2 "MountingHole:MountingHole_3.2mm_M3" H 2250 6600 50  0001 C CNN
+F 3 "~" H 2250 6600 50  0001 C CNN
+	1    2250 6600
+	1    0    0    -1
+$EndComp
+$Comp
+L Mechanical:MountingHole H4
+U 1 1 5F93C152
+P 2250 6900
+F 0 "H4" H 2350 6946 50  0000 L CNN
+F 1 "MountingHole" H 2350 6855 50  0000 L CNN
+F 2 "MountingHole:MountingHole_3.2mm_M3" H 2250 6900 50  0001 C CNN
+F 3 "~" H 2250 6900 50  0001 C CNN
+	1    2250 6900
+	1    0    0    -1
+$EndComp
 $EndSCHEMATC
