File: KiCAD/Antilog_NPNO_PCB Ver.1.2/Antilog_NPNO_PCB.kicad_pcb (KiCad board)
At the start: 2 copper layers, 88.9 x 61 mm, 47 parts, among them J1 PWR_IN, J10 I_SINK, J2 TP_GND, J3 MOD, J4 COUARSE, J5 CV, J6 MOD2, J7 MSTR_OUT, J8 TP_ADJ, J9 VREF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

Commit message: Updated: Ver.1.2 PCB Design
Parts:
- added G***: LOGO, myfootprint:Silk_PNPN_Manufactory_600dpi, F.Cu at (158.0, 97.0)
- moved R14 22.2 mm to (146.1, 74.9), turned to 270 degrees
- moved J8 21.6 mm to (168.9, 74.9)
- moved J6 20.7 mm to (134.6, 120.7)
- moved R8 20.5 mm to (134.6, 106.7)
- moved C5 20.4 mm to (149.9, 97.8), turned to 180 degrees
- moved R13 20.1 mm to (131.4, 87.6), turned to 270 degrees
- moved RV4 14.0 mm to (151.1, 86.4)
- moved H4 13.3 mm to (182.4, 122.7)
- moved H2 12.7 mm to (182.4, 71.6)
- moved J2 11.7 mm to (166.4, 123.2)
- moved R17 11.5 mm to (145.4, 87.0)
- moved J3 10.9 mm to (124.5, 120.7)
- moved J4 10.9 mm to (157.5, 120.7)
- moved R4 10.5 mm to (151.8, 114.3)
- moved R10 10.5 mm to (154.9, 106.7)
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Connections:
- U1 pad 1: Net-(C5-Pad1) -> Net-(R13-Pad1)
- U1 pad 2: Net-(C5-Pad2) -> Net-(R10-Pad1)
- U1 pad 6: Net-(R10-Pad1) -> Net-(C5-Pad2)
- U1 pad 7: Net-(R13-Pad1) -> Net-(C5-Pad1)
Routing:
- net +12V: track 0.00 -> 164.6 mm
- net -12V: track 0.00 -> 96.0 mm
- net Net-(R10-Pad1): track 0.00 -> 76.3 mm
- net Net-(C5-Pad2): track 0.00 -> 68.2 mm
- net Net-(R13-Pad1): track 0.00 -> 38.4 mm
- net Net-(Q2-Pad2): track 0.00 -> 32.1 mm
- net Net-(Q1-Pad1): track 0.00 -> 22.0 mm
- net Net-(J7-Pad1): track 0.00 -> 20.1 mm
- net Net-(J9-Pad1): track 0.00 -> 14.2 mm
- net Net-(J3-Pad1): track 0.00 -> 13.9 mm
- net Net-(Q1-Pad3): track 0.00 -> 13.5 mm
- net Net-(J8-Pad1): track 0.00 -> 13.0 mm
- net Net-(C5-Pad1): track 0.00 -> 9.20 mm
- net Net-(R14-Pad2): track 0.00 -> 6.66 mm
- net Net-(J4-Pad3): track 0.00 -> 6.65 mm
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- added copper zone on B.Cu, net GND
- added copper zone on F.Cu, net GND
Other:
- board size 88.9 x 61 mm -> 76.2 x 57.2 mm
- board text added: "+12V"
- board text added: "- COUARSE +"
- board text added: "ADJ"
- board text added: "Antilog NPNO Ver.1.2"
- board text added: "FINE"
- board text added: "G CV"
- board text added: "G MOD"
- board text added: "G MOD2"
- board text added: "GND"
- board text added: "I_SINK G"
- board text added: "MOD_LVL"
- board text added: "MSTR_OUT"
- board text added: "PWR_IN"
- board text added: "SCALE"
- board text added: "TP_ADJ"
- board text added: "V+ G V-"
- board text added: "VREF G"
- board text added: "https://dad8893.blogspot.com/"
