File: KiCAD/Antilog_NPNO_PCB Ver.1.2/Antilog_NPNO_PCB.sch (KiCad schematic (older format))
At the start: 47 parts, among them J1 PWR_IN, J10 I_SINK, J2 TP_GND, J3 MOD, J4 COUARSE, J5 CV, J6 MOD2, J7 MSTR_OUT, J8 TP_ADJ, J9 VREF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

Commit message: Updated: Ver.1.2 PCB Design
Connections:
- net GND: now also U1.3 (+), U1.5 (+); no longer U1.3 (+), U1.5 (+)
- net at R10.1, R11.1, R12.2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: now also U1.2 (-); no longer U1.6 (-)
- net at R13.1, RV4.2, RV4.3: now also U1.1; no longer U1.7
- net at C5.1, R17.2: now also U1.7; no longer U1.1
- net at C5.2, Q1.2 (C), R16.2: now also U1.6 (-); no longer U1.2 (-)
Changed lines of the file:
@@
 Sheet 1 1
 Title "Antilog_NPNO"
-Date "2020-12-14"
+Date "2020-12-29"
 Rev "Ver. 1.2"
 Comp "PNPN Manufactory"
@@
 $Comp
 L Amplifier_Operational:TL072 U1
-U 2 1 5F8E2874
+U 1 1 5F8E2874
 P 6900 4150
 F 0 "U1" H 6550 4550 50  0000 C CNN
@@
 F 2 "Package_DIP:DIP-8_W7.62mm_Socket" H 6900 4150 50  0001 C CNN
 F 3 "http://www.ti.com/lit/ds/symlink/tl071.pdf" H 6900 4150 50  0001 C CNN
-	2    6900 4150
+	1    6900 4150
 	1    0    0    -1
 $EndComp
@@
 $Comp
 L Amplifier_Operational:TL072 U1
-U 1 1 5F8E9E6F
+U 2 1 5F8E9E6F
 P 8950 5100
 F 0 "U1" H 8950 5467 50  0000 C CNN
@@
 F 2 "Package_DIP:DIP-8_W7.62mm_Socket" H 8950 5100 50  0001 C CNN
 F 3 "http://www.ti.com/lit/ds/symlink/tl071.pdf" H 8950 5100 50  0001 C CNN
-	1    8950 5100
+	2    8950 5100
 	1    0    0    -1
 $EndComp
